File: pcb/mad cat.kicad_pcb (KiCad board)
At the start: 2 copper layers, 361.9 x 147 mm, 259 parts, among them J1 Conn_01x04, J2 Conn_02x03_Odd_Even, SW0,0 ESC, SW0,1 ESC/F1, SW0,10 F9, SW0,10-1 F10, SW0,11 F10, SW0,11-1 F11, SW0,12 F11, SW0,12-1 F12, SW0,13 F12/PRT, SW0,14 INS, SW0,15 HOME, SW0,16 PGUP, SW0,2 F1, SW0,2-1 F2, SW0,3 F2, SW0,3-1 F3, SW0,4 F3, SW0,4-1 F4, SW0,5 F4, SW0,5-1 F5, SW0,6 F5, SW0,6-1 F6, SW0,7 F6, SW0,7-1 F7, SW0,8 F7, SW0,8-1 F8, SW0,9 F8, SW0,9-1 F9, SW1,0 PF1, SW1,1 TILDE, SW1,10 9, SW1,11 0, SW1,12 -, SW1,13 =, SW1,14 BACKSPACE, SW1,14-1 S_BS_L, SW1,15 END, SW1,16 PGDN, SW1,2 1, SW1,3 2, SW1,4 3, SW1,5 4, SW1,6 5, SW1,7 6, SW1,8 7, SW1,9 8, SW2,0 PF2, SW2,1 TAB, SW2,10 O, SW2,11 P, SW2,12 [, SW2,13 ], SW2,14 \, SW2,15 S_BS_R, SW2,16 PRT, SW2,2 Q, SW2,3 W, SW2,4 E, SW2,5 R, SW2,6 T, SW2,7 Y, SW2,8 U, SW2,9 I, SW3,0 PF3, SW3,1 CAPS, SW3,1-1 ST_CAPS, SW3,10 L, SW3,11 COLONS, SW3,12 QUOTE, SW3,13 ISO_#, SW3,14 ENT, SW3,14-1 ISO_ENT, SW3,15 DEL, SW3,15-1 DEL, SW3,16 NP_ENT, SW3,16-1 1U_ENT, SW3,2 A, SW3,3 S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

Commit message: "finished" traces
Parts:
- D1, D10, D11, D12, D13, D14, D15, D16, D17, D18, D19, D2, D20, D21, D22, D23, D24, D25, D26, D27, D28, D29, D3, D30, D31, D32, D33, D34, D35, D36, D37, D38, D39, D4, D40, D41, D42, D43, D44, D45, D46, D47, D48, D49, D5, D50, D51, D52, D53, D54, D55, D56, D57, D58, D59, D6, D60, D61, D62, D63, D64, D65, D66, D67, D68, D69, D7, D70, D71, D72, D73, D74, D75, D76, D77, D78, D79, D8, D80, D81, D82, D83, D84, D85, D86, D87, D88, D89, D9, D90, D91, D92, D93, D94, D95: footprint Diode_SMD:D_SOD-123 -> keebs:D_SOD-123proto
- moved C12 239.6 mm to (351.7, 71.8), turned to 90 degrees
- moved C13 235.1 mm to (342.0, 60.2), turned to 90 degrees
- moved R9 234.5 mm to (349.9, 70.2), turned to 90 degrees
- moved R10 232.2 mm to (343.9, 62.8), turned to 180 degrees
- moved R7 167.6 mm to (6.80, 16.2), turned to 180 degrees
- moved R8 166.5 mm to (14.5, 13.4), turned to 180 degrees
- moved C10 166.1 mm to (6.80, 14.3)
- moved C11 165.1 mm to (14.5, 11.7)
- moved C1 0.93 mm to (119.8, 108.9)
- moved R1 0.14 mm to (125.7, 121.3)
- turned EC2-1 to 335 degrees
Routing:
- net GND: track 252.3 -> 684.7 mm, vias 3 -> 6
- net /enc+: track 263.0 -> 527.1 mm, vias 3 -> 7
- net /RES: track 0.00 -> 248.7 mm, vias 0 -> 2
- net /r5: track 148.5 -> 357.4 mm, vias 4 -> 5
- net /r0: track 317.5 -> 455.4 mm, vias 0 -> 4
- net /c13: track 190.8 -> 327.6 mm
- net Net-(LED1-Pad2): track 183.3 -> 267.2 mm
- net VCC: track 224.8 -> 298.5 mm, vias 4 -> 9
- net /r1: track 346.9 -> 420.3 mm, vias 4 -> 6
- net /enc-: track 466.9 -> 523.3 mm, vias 3 -> 6
- net /c12: track 225.6 -> 274.6 mm
- net /c3: track 146.0 -> 194.1 mm
- net /c0: track 216.0 -> 257.2 mm
- net /c4: track 108.0 -> 149.0 mm, vias 0 -> 1
- net /c1: track 261.0 -> 301.2 mm, vias 1 -> 2
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Other:
- outline, holes or cut-outs redrawn

Commit message: even more compat, generating gerbers
Parts:
- added SW5,2-2: ALT, MX_SMK_2:MX_SMK_150, F.Cu at (68.3, 111.1)
- added SW5,7-3: 7 SPACE, MX_SMK_2:MX_SMK_700_stabflip, F.Cu at (149.2, 111.1)
- D1, D10, D11, D12, D13, D14, D15, D16, D17, D18, D19, D2, D20, D21, D22, D23, D24, D25, D26, D27, D28, D29, D3, D30, D31, D32, D33, D34, D35, D36, D37, D38, D39, D4, D40, D41, D42, D43, D44, D45, D46, D47, D48, D49, D5, D50, D51, D52, D53, D54, D55, D56, D57, D58, D59, D6, D60, D61, D62, D63, D64, D65, D66, D67, D68, D69, D7, D70, D71, D72, D73, D74, D75, D76, D77, D78, D79, D8, D80, D81, D82, D83, D84, D85, D86, D87, D88, D89, D9, D90, D91, D92, D93, D94, D95: footprint keebs:D_SOD-123proto -> Diode_SMD:D_SOD-123
- moved D89 1.72 mm to (146.5, 115.0)
Routing:
- net /c11: track 264.0 -> 244.7 mm
- net GND: track 684.7 -> 699.0 mm, vias 6 -> 7
- net /c7: track 169.0 -> 183.2 mm
- net Net-(D87-Pad2): track 11.0 -> 24.2 mm
- net /c12: track 274.6 -> 266.5 mm
- net Net-(D51-Pad2): track 31.2 -> 38.6 mm
- net /c2: track 290.3 -> 285.3 mm
- net /r5: track 357.4 -> 362.1 mm
- net Net-(D89-Pad2): track 18.6 -> 22.8 mm
- net /c13: track 327.6 -> 331.6 mm
- net /c16: track 358.9 -> 360.1 mm
Other:
- outline, holes or cut-outs redrawn

Commit message: editing flex cuts
Routing:
- net /c13: track 331.6 -> 344.8 mm
- net /c2: track 285.3 -> 295.7 mm
- net /c14: track 347.6 -> 353.4 mm
- net /RES: track 248.7 -> 245.0 mm
- net /c0: track 257.2 -> 254.7 mm
- net /r5: track 362.1 -> 364.2 mm
- net /c12: track 266.5 -> 267.8 mm
- net /c3: track 194.6 -> 193.6 mm
- net /enc-: track 523.3 -> 522.4 mm
- net /enc+: track 527.1 -> 526.5 mm
Other:
- outline, holes or cut-outs redrawn

Commit message: Updating a lot
Parts:
- moved C3 7.00 mm to (132.5, 115.6), turned to 225 degrees
- moved C1 6.00 mm to (113.8, 108.9)
- moved C2 6.00 mm to (128.7, 103.2)
- moved C4 6.00 mm to (127.5, 121.5)
- moved C5 6.00 mm to (116.5, 117.5)
- moved C6 6.00 mm to (115.2, 120.5)
- moved C7 6.00 mm to (113.0, 106.5)
- moved C8 6.00 mm to (118.9, 101.9)
- moved C9 6.00 mm to (129.0, 120.0)
- moved R1 6.00 mm to (119.7, 121.3)
- moved R2 6.00 mm to (118.6, 120.2)
- moved U1 6.00 mm to (124.0, 112.0)
- moved Y1 6.00 mm to (116.7, 104.3)
- moved D89 2.50 mm to (144.5, 113.5), turned to 0 degrees
Routing:
- net /c13: track 344.8 -> 369.4 mm
- net /c10: track 233.1 -> 252.9 mm
- net /c3: track 193.6 -> 209.9 mm
- net /r5: track 364.2 -> 375.5 mm, vias 5 -> 4
- net /c4: track 149.0 -> 157.5 mm
- net /c14: track 353.4 -> 361.3 mm
- net /c15: track 364.5 -> 372.3 mm
- net /c12: track 267.8 -> 275.3 mm
- net /c11: track 244.7 -> 252.2 mm
- net /c16: track 360.1 -> 367.3 mm
- net /c1: track 301.0 -> 294.5 mm
- net Net-(LED1-Pad2): track 267.2 -> 273.4 mm
- net /c9: track 186.7 -> 192.7 mm
- net /c8: track 165.5 -> 171.5 mm
- net /c7: track 183.2 -> 189.2 mm
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Other:
- outline, holes or cut-outs redrawn

Commit message: new flex cuts
Parts:
- added SW4,15-1: Extra 1u, MX_SMK_2:MX_SMK_100, F.Cu at (333.4, 92.1)
- moved R8 0.22 mm to (14.6, 13.2)
- moved C11 0.22 mm to (14.6, 11.5)
- turned EC1 to 114.5 degrees
Routing:
- net Net-(D84-Pad2): track 6.64 -> 13.6 mm
- net /c15: track 372.3 -> 378.8 mm
- net /enc+: track 524.4 -> 525.9 mm
- net /enc-: track 519.2 -> 520.6 mm
- net /r5: track 375.5 -> 376.9 mm, vias 4 -> 5
- net /c0: track 249.1 -> 250.5 mm
- net /c16: track 367.3 -> 368.4 mm
Other:
- outline, holes or cut-outs redrawn

Commit message: redoing in mx only, adding trimpot for led
Parts:
- added POT1: TC33X-2-103E, digikey-footprints:Trimpot_3.8mmx3.6mm_TC33X-2-103E, B.Cu at (317.5, 31.5)
- LED1: footprint keebs:LED_D1.8mm_W3.3mm_H2.4mm_CENTERED -> keebs:LED_0805_lightpipe
- R5: value >390 -> 440
- SW0,0, SW0,1, SW0,10, SW0,10-1, SW0,11, SW0,11-1, SW0,12, SW0,12-1, SW0,13, SW0,14, SW0,15, SW0,16, SW0,2, SW0,2-1, SW0,3, SW0,3-1, SW0,4, SW0,4-1, SW0,5, SW0,5-1, SW0,6, SW0,6-1, SW0,7, SW0,7-1, SW0,8, SW0,8-1, SW0,9, SW0,9-1, SW1,0, SW1,1, SW1,10, SW1,11, SW1,12, SW1,13, SW1,14-1, SW1,15, SW1,16, SW1,2, SW1,3, SW1,4, SW1,5, SW1,6, SW1,7, SW1,8, SW1,9, SW2,0, SW2,10, SW2,11, SW2,12, SW2,13, SW2,15, SW2,16, SW2,2, SW2,3, SW2,4, SW2,5, SW2,6, SW2,7, SW2,8, SW2,9, SW3,0, SW3,10, SW3,11, SW3,12, SW3,13, SW3,16-1, SW3,2, SW3,3, SW3,4, SW3,5, SW3,6, SW3,7, SW3,8, SW3,9, SW4,0, SW4,10, SW4,11, SW4,12, SW4,14, SW4,14-1, SW4,15, SW4,15-1, SW4,2, SW4,3, SW4,4, SW4,5, SW4,6, SW4,7, SW4,8, SW4,9, SW5,0, SW5,0-1, SW5,12, SW5,13-1, SW5,14, SW5,15, SW5,16, SW5,2: footprint MX_SMK_2:MX_SMK_100 -> MX_SMK_2:MX_100
- SW1,14, SW3,15, SW3,15-1, SW3,16, SW5,16-1: footprint MX_SMK_2:MX_SMK_200 -> MX_SMK_2:MX_200
- SW2,1, SW2,14, SW5,1, SW5,11, SW5,12-1, SW5,12-2, SW5,13, SW5,2-2, SW5,3: footprint MX_SMK_2:MX_SMK_150 -> MX_SMK_2:MX_150
- SW3,1, SW4,13: footprint MX_SMK_2:MX_SMK_175 -> MX_SMK_2:MX_175
- SW3,1-1, SW4,1-1, SW5,1-1, SW5,2-1, SW5,3-1: footprint MX_SMK_2:MX_SMK_125 -> MX_SMK_2:MX_125
- SW3,14, SW4,1: footprint MX_SMK_2:MX_SMK_225 -> MX_SMK_2:MX_225
- SW3,14-1: footprint MX_SMK_2:MX_SMK_ISO_stabflip -> MX_SMK_2:MX_ISO_stabflip
- SW4,13-1: footprint MX_SMK_2:MX_SMK_275 -> MX_SMK_2:MX_275
- SW5,7: footprint MX_SMK_2:MX_SMK_600_stabflip -> MX_SMK_2:MX_600_stabflip
- SW5,7-1: footprint MX_SMK_2:MX_SMK_625_stabflip -> MX_SMK_2:MX_625_stabflip
- SW5,7-2, SW5,7-3: footprint MX_SMK_2:MX_SMK_700_stabflip -> MX_SMK_2:MX_700_stabflip
- moved R5 12.3 mm to (315.7, 36.0), turned to 270 degrees
- moved R8 3.01 mm to (17.6, 13.0)
- moved C11 3.00 mm to (17.6, 11.4)
- moved C10 1.78 mm to (8.20, 15.4)
- moved C1 1.43 mm to (112.7, 109.9)
- moved R7 1.30 mm to (7.50, 17.3)
- turned EC1 to 120 degrees
- turned LED1 to 0 degrees
Connections:
- LED1 pad 1: Net-(LED1-Pad1) -> GND
- R5 pad 1: GND -> Net-(POT1-Pad1)
- R5 pad 2: Net-(LED1-Pad1) -> Net-(R5-Pad2)
- U1 pad 33: Net-(LED1-Pad2) -> Net-(R5-Pad2)
Routing:
- net Net-(LED1-Pad2): track 273.4 -> 6.30 mm, vias 2 -> 1
- net Net-(R5-Pad2): track 0.00 -> 263.8 mm, vias 0 -> 2
- net /c10: track 252.9 -> 279.5 mm
- net /c11: track 252.2 -> 272.6 mm
- net /c3: track 209.9 -> 190.4 mm, vias 0 -> 1
- net /RES: track 239.3 -> 220.8 mm, vias 2 -> 3
- net /enc-: track 520.6 -> 504.0 mm, vias 6 -> 4
- net /c7: track 189.2 -> 172.6 mm
- net /enc+: track 525.9 -> 541.2 mm, vias 7 -> 4
- net /c14: track 361.3 -> 347.5 mm
- net Net-(D32-Pad2): track 27.9 -> 16.2 mm
- net /c2: track 291.8 -> 302.4 mm
- net /c4: track 157.5 -> 147.3 mm
- net /c12: track 275.3 -> 284.1 mm
- net GND: track 704.7 -> 713.0 mm, vias 5 -> 12
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Other:
- outline, holes or cut-outs redrawn

Commit message: fixed silk, created gerbers
Parts:
- added SW1,0-1: PF1, MX_SMK_2:MX_100, F.Cu at (9.53, 41.3)
- added SW2,0-1: PF2, MX_SMK_2:MX_100, F.Cu at (9.53, 60.3)
- added SW3,0-1: PF3, MX_SMK_2:MX_100, F.Cu at (9.53, 79.4)
- added SW4,0-1: PF4, MX_SMK_2:MX_100, F.Cu at (9.53, 98.4)
- moved D18 11.6 mm to (18.0, 40.4)
- moved D35 11.6 mm to (18.0, 59.5)
- moved D52 11.6 mm to (18.0, 78.5)
- moved D69 11.6 mm to (18.0, 97.5)
Routing:
- net /r3: track 405.6 -> 393.5 mm
- net /r4: track 341.0 -> 328.9 mm
- net Net-(D18-Pad2): track 6.64 -> 18.6 mm
- net Net-(D69-Pad2): track 6.64 -> 18.6 mm
- net Net-(D52-Pad2): track 6.64 -> 18.6 mm
- net Net-(D35-Pad2): track 6.64 -> 18.6 mm
- net /r1: track 424.0 -> 412.4 mm
- net /r2: track 406.3 -> 394.7 mm
- net /c0: track 247.2 -> 249.5 mm

Commit message: via stitching lol
Parts:
- D1, D10, D11, D12, D13, D14, D15, D16, D17, D18, D19, D2, D20, D21, D22, D23, D24, D25, D26, D27, D28, D29, D3, D30, D31, D32, D33, D34, D35, D36, D37, D38, D39, D4, D40, D41, D42, D43, D44, D45, D46, D47, D48, D49, D5, D50, D51, D52, D53, D54, D55, D56, D57, D58, D59, D6, D60, D61, D62, D63, D64, D65, D66, D67, D68, D69, D7, D70, D71, D72, D73, D74, D75, D76, D77, D78, D79, D8, D80, D81, D82, D83, D84, D85, D86, D87, D88, D89, D9, D90, D91, D92, D93, D94, D95: footprint Diode_SMD:D_SOD-123 -> keebs:D_SOD-123proto
Routing:
- net GND: track 713.0 -> 245.5 mm, vias 12 -> 5723
- net /c2: track 302.4 -> 271.1 mm
- net /r5: track 384.0 -> 404.6 mm
- net /c3: track 190.4 -> 176.1 mm
- net /c4: track 147.3 -> 160.6 mm
- net /c8: track 169.7 -> 179.0 mm
- net /c0: track 249.5 -> 242.4 mm
- net /RES: track 220.8 -> 216.3 mm
- net /enc+: track 541.2 -> 538.6 mm
- net /enc-: track 504.0 -> 501.4 mm
- net /c1: track 298.0 -> 295.6 mm
- added copper zone on F.Cu, net GND
Other:
- outline, holes or cut-outs redrawn
