File: pcb/mad cat.kicad_pcb (KiCad board)
At the start: 2 copper layers, 361.9 x 143 mm, 274 parts, among them J1 Conn_01x04, J2 Conn_02x03_Odd_Even, SW0,0 ESC, SW0,1 ESC/F1, SW0,10 F9, SW0,10-1 F10, SW0,11 F10, SW0,11-1 F11, SW0,12 F11, SW0,12-1 F12, SW0,13 F12/PRT, SW0,14 INS, SW0,15 HOME, SW0,16 PGUP, SW0,2 F1, SW0,2-1 F2, SW0,3 F2, SW0,3-1 F3, SW0,4 F3, SW0,4-1 F4, SW0,5 F4, SW0,5-1 F5, SW0,6 F5, SW0,6-1 F6, SW0,7 F6, SW0,7-1 F7, SW0,8 F7, SW0,8-1 F8, SW0,9 F8, SW0,9-1 F9, SW1,0 PF1, SW1,0-1 PF1, SW1,1 TILDE, SW1,10 9, SW1,11 0, SW1,12 -, SW1,13 =, SW1,14 BACKSPACE, SW1,14-1 S_BS_L, SW1,15 END, SW1,15-1 HOME, SW1,16 PGDN, SW1,16-1 PGUP, SW1,2 1, SW1,3 2, SW1,4 3, SW1,5 4, SW1,6 5, SW1,7 6, SW1,8 7, SW1,9 8, SW2,0 PF2, SW2,0-1 PF2, SW2,1 TAB, SW2,10 O, SW2,11 P, SW2,12 [, SW2,13 ], SW2,14 \, SW2,15 S_BS_R, SW2,16 PRT, SW2,2 Q, SW2,3 W, SW2,4 E, SW2,5 R, SW2,6 T, SW2,7 Y, SW2,8 U, SW2,9 I, SW3,0 PF3, SW3,0-1 PF3, SW3,1 CAPS, SW3,1-1 ST_CAPS, SW3,10 L, SW3,11 COLONS, SW3,12 QUOTE, SW3,13 ISO_#, SW3,14 ENT, SW3,14-1 ISO_ENT, SW3,15 DEL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

Commit message: starting on pre production
Parts:
- removed the G*** at (201.0, 111.1)
- EC1, EC2: footprint keebs:EC11E -> crokto:EC11E
- H1, H10, H2, H3, H4, H5, H6, H7, H8, H9: footprint keebs:m2.5_pad_via -> crokto:m2.5_pad_via
- J2: footprint keebs:PinHeader_2x03_P1.27mm_Vertical_center -> crokto:PinHeader_2x03_P1.27mm_Vertical_center
- SW5,7-1: footprint MX_SMK_2:MX_600_stabflip3 -> MX_SMK_2:MX_600_stabflip_3
- moved D90 8.97 mm to (141.6, 105.8), turned to 90 degrees
- turned D51 to 90 degrees
Routing:
- net /r5: track 405.6 -> 398.6 mm
- net Net-(D97-Pad2): track 36.2 -> 32.2 mm
- net Net-(D51-Pad2): track 15.2 -> 18.8 mm
- net /r2: track 412.6 -> 414.4 mm
- net GND: track 291.8 -> 293.6 mm, vias 71 -> 81
- net /enc-: track 516.9 -> 518.1 mm
- net /c1: track 286.7 -> 287.8 mm
- net /enc+: track 535.9 -> 537.1 mm
- net /c0: track 240.7 -> 241.9 mm
- net Net-(D90-Pad2): track 26.0 -> 25.1 mm
Other:
- rule trace_min: 0.2032 -> 0.2
- board text added: "by Chris Grossman"
- board text removed: "Proto by Chris Grossman"

Commit message: prepared for pcba
Parts:
- removed G***: LOGO, logo:metamechs logo half
- added LOGO1: MountingHole, logo:metamechs logo half, B.Cu at (201.0, 111.0)
- RST1: footprint Button_Switch_SMD:SW_SPST_SKQG_WithStem -> crokto:TS-1187A-B-A-B
- SW4,13: footprint MX_SMK_2:MX_175 -> MX_SMK_2:MX_175_labeled
- SW4,13-1: footprint MX_SMK_2:MX_275 -> MX_SMK_2:MX_275_labeled
- SW5,1, SW5,11-1, SW5,3: footprint MX_SMK_2:MX_150 -> MX_SMK_2:MX_150_labeled
- SW5,1-1, SW5,2-1, SW5,3-1: footprint MX_SMK_2:MX_125 -> MX_SMK_2:MX_125_labeled
- SW5,11, SW5,2: footprint MX_SMK_2:MX_100 -> MX_SMK_2:MX_100_labeled
- Y1: footprint Crystal:Crystal_SMD_SeikoEpson_FA238-4Pin_3.2x2.5mm -> Crystal:Crystal_SMD_SeikoEpson_TSX3225-4Pin_3.2x2.5mm
Other:
- board text added: "JLCJLCJLCJLC"

Commit message: edited LED circuit, flipped stabs
Parts:
- added ESD1: PRTR5V0U2X, Package_TO_SOT_SMD:SOT-143, B.Cu at (21.6, 32.0)
- added PTC1: 500mA, Fuse:Fuse_0805_2012Metric, B.Cu at (23.9, 37.3)
- C5: value 1u -> 10u
- R5: value 440 -> 510
- SW5,7: footprint MX_SMK_2:MX_625_stabflip -> MX_SMK_2:MX_625_nonflipped
- SW5,7-1: footprint MX_SMK_2:MX_600_stabflip_3 -> MX_SMK_2:MX_600_unflipped_3
- moved POT1 0.96 mm to (318.5, 41.5), turned to 180 degrees
- moved C7 0.64 mm to (113.4, 107.0)
Connections:
- J1 pad 4: VCC -> vbus
- POT1 pad 1: Net-(POT1-Pad1) -> Net-(LED1-Pad2)
- POT1 pad 3: GND -> Net-(POT1-Pad3)
- R5 pad 1: Net-(POT1-Pad1) -> Net-(POT1-Pad3)
Routing:
- net GND: track 293.4 -> 392.5 mm, vias 81 -> 80
- net vbus: track 0.00 -> 16.6 mm, vias 0 -> 4
- net /RES: track 214.6 -> 218.1 mm
- net VCC: track 293.4 -> 290.1 mm
- net Net-(POT1-Pad3): track 0.00 -> 3.05 mm
- net Net-(POT1-Pad1): track 2.71 -> 0.00 mm
- net Net-(LED1-Pad2): track 15.5 -> 17.5 mm
- net Net-(R5-Pad2): track 268.5 -> 270.3 mm
- net /D-: track 201.4 -> 202.6 mm
- net /D+: track 201.1 -> 201.8 mm
- net /c1: track 287.8 -> 288.3 mm, vias 2 -> 1

Commit message: new edge cuts
Parts:
- RST1: moved to F.Cu
- SW5,7: footprint MX_SMK_2:MX_625_nonflipped -> MX_SMK_2:MX_625_stabflip
- SW5,7-1: footprint MX_SMK_2:MX_600_unflipped_3 -> MX_SMK_2:MX_600_stabflip_3
- moved RST1 198.1 mm to (190.0, 111.1)
- moved R6 196.2 mm to (184.4, 108.3)
- moved C10 7.06 mm to (13.0, 21.0), turned to 90 degrees
- moved C11 5.44 mm to (19.5, 16.5)
- moved R7 4.83 mm to (11.1, 21.0), turned to 270 degrees
- moved R8 2.60 mm to (19.5, 14.8)
Routing:
- net GND: track 392.5 -> 275.0 mm, vias 80 -> 104
- net /RES: track 218.1 -> 319.9 mm, vias 3 -> 5
- net VCC: track 290.1 -> 343.1 mm, vias 8 -> 9
- net /r4: track 378.9 -> 367.3 mm
- net /c14: track 382.1 -> 378.2 mm
- net /r0: track 446.2 -> 449.3 mm, vias 4 -> 2
- net /enc-: track 518.1 -> 515.0 mm
- net /c12: track 339.0 -> 336.4 mm
- net /c11: track 290.7 -> 288.3 mm
- net /enc+: track 537.1 -> 539.4 mm
- net /c15: track 420.7 -> 418.8 mm
- net /c16: track 401.7 -> 400.0 mm
- net Net-(D97-Pad2): track 32.2 -> 33.8 mm
- net /c13: track 356.3 -> 355.1 mm
- net Net-(D67-Pad2): track 38.4 -> 39.6 mm
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Other:
- board size 361.9 x 143 mm -> 360.9 x 142 mm

Commit message: tweaked tracks
Parts:
- moved D1 4.44 mm to (6.85, 17.5)
- moved D74 3.00 mm to (108.9, 96.1)
- moved D2 2.00 mm to (27.9, 14.5)
- moved D79 1.00 mm to (203.1, 99.1)
- moved R6 0.43 mm to (184.0, 108.5)
Routing:
- net /r0: track 449.3 -> 445.3 mm
- net /c15: track 418.8 -> 421.9 mm
- net Net-(D74-Pad2): track 10.1 -> 7.14 mm
- net Net-(D1-Pad2): track 14.7 -> 12.4 mm
- net /enc-: track 515.0 -> 512.9 mm, vias 4 -> 2
- net Net-(D2-Pad2): track 9.71 -> 8.14 mm
- net /enc+: track 539.4 -> 537.9 mm, vias 4 -> 2
- net /r5: track 398.0 -> 396.9 mm, vias 5 -> 7
- net /c3: track 177.2 -> 177.9 mm, vias 1 -> 0
- net /RES: track 319.9 -> 320.4 mm
- net /c14: vias 1 -> 0
- net GND: vias 104 -> 99
Other:
- outline, holes or cut-outs redrawn
