File: pcb/mad cat.sch (KiCad schematic (older format))
At the start: 257 parts, among them J1 Conn_01x04, J2 Conn_02x03_Odd_Even, SW0,0 ESC, SW0,1 ESC/F1, SW0,10 F9, SW0,10-1 F10, SW0,11 F10, SW0,11-1 F11, SW0,12 F11, SW0,12-1 F12, SW0,13 F12/PRT, SW0,14 INS, SW0,15 HOME, SW0,16 PGUP, SW0,2 F1, SW0,2-1 F2, SW0,3 F2, SW0,3-1 F3, SW0,4 F3, SW0,4-1 F4, SW0,5 F4, SW0,5-1 F5, SW0,6 F5, SW0,6-1 F6, SW0,7 F6, SW0,7-1 F7, SW0,8 F7, SW0,8-1 F8, SW0,9 F8, SW0,9-1 F9, SW1,0 PF1, SW1,0-1 PF1, SW1,1 TILDE, SW1,10 9, SW1,11 0, SW1,12 -, SW1,13 =, SW1,14 BACKSPACE, SW1,14-1 S_BS_L, SW1,15 END, SW1,16 PGDN, SW1,2 1, SW1,3 2, SW1,4 3, SW1,5 4, SW1,6 5, SW1,7 6, SW1,8 7, SW1,9 8, SW2,0 PF2, SW2,0-1 PF2, SW2,1 TAB, SW2,10 O, SW2,11 P, SW2,12 [, SW2,13 ], SW2,14 \\, SW2,15 S_BS_R, SW2,16 PRT, SW2,2 Q, SW2,3 W, SW2,4 E, SW2,5 R, SW2,6 T, SW2,7 Y, SW2,8 U, SW2,9 I, SW3,0 PF3, SW3,0-1 PF3, SW3,1 CAPS, SW3,1-1 ST_CAPS, SW3,10 L, SW3,11 COLONS, SW3,12 QUOTE, SW3,13 ISO_#, SW3,14 ENT, SW3,14-1 ISO_ENT, SW3,15 DEL, SW3,15-1 DEL, SW3,16 NP_ENT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

Commit message: added support for 2 1us on del
Parts:
- added D84: D, Diode_SMD:D_SOD-123, symbol keyboard_parts:D
- added SW3,15-2, SW3,15-3: DEL, MX_SMK_2:MX_100, symbol keyboard_parts:SW_PUSH
- added SW4,15, SW4,15-1: Extra 1u, MX_SMK_2:MX_100, symbol keyboard_parts:SW_PUSH
- POT1: symbol dk_Trimmer-Potentiometers:TC33X-2-103E -> mad-cat-rescue:TC33X-2-103E-dk_Trimmer-Potentiometers
- renumbered D84 to D85, D85 to D86, D86 to D87, D87 to D88, D88 to D89, D89 to D90, D90 to D91, D91 to D92, D92 to D93, D93 to D94, D94 to D95, D95 to D96, SW4,15 to SW4,16, SW4,15-1 to SW4,16-1
Connections:
- net c15: now also SW3,15-2.2, SW3,15-3.2, SW4,15-1.2, SW4,15.2; no longer SW4,16-1.2, SW4,16.2
- net c16: now also SW4,16-1.2, SW4,16.2
- net r4: now also D84.1
- net at D67.2, SW3,15-1.1, SW3,15.1: now also SW3,15-2.1, SW3,15-3.1
- new net: D84.2, SW4,15-1.1, SW4,15.1
Other:
- moved on the sheet: D85, SW3,15-1, SW4,16, SW4,16-1
Changed lines of the file:
@@
 $EndComp
 $Comp
-L keyboard_parts:D D85
+L keyboard_parts:D D86
 U 1 1 5CBB743B
 P 750 4200
-F 0 "D85" H 800 4000 60  0000 R CNN
+F 0 "D86" H 800 4000 60  0000 R CNN
 F 1 "D" V 900 4150 60  0001 C CNN
 F 2 "Diode_SMD:D_SOD-123" H 750 4200 60  0001 C CNN
@@
 $EndComp
 $Comp
-L keyboard_parts:D D86
+L keyboard_parts:D D87
 U 1 1 5CBBC11C
 P 1500 4200
-F 0 "D86" H 1550 4000 60  0000 R CNN
+F 0 "D87" H 1550 4000 60  0000 R CNN
 F 1 "D" V 1650 4150 60  0001 C CNN
 F 2 "Diode_SMD:D_SOD-123" H 1500 4200 60  0001 C CNN
@@
 $EndComp
 $Comp
-L keyboard_parts:D D87
+L keyboard_parts:D D88
 U 1 1 5CBBED3A
 P 2250 4200
-F 0 "D87" H 2300 4000 60  0000 R CNN
+F 0 "D88" H 2300 4000 60  0000 R CNN
 F 1 "D" V 2400 4150 60  0001 C CNN
 F 2 "Diode_SMD:D_SOD-123" H 2250 4200 60  0001 C CNN
@@
 $EndComp
 $Comp
-L keyboard_parts:D D88
+L keyboard_parts:D D89
 U 1 1 5CBBED99
 P 3000 4200
-F 0 "D88" H 3050 4000 60  0000 R CNN
+F 0 "D89" H 3050 4000 60  0000 R CNN
 F 1 "D" V 3150 4150 60  0001 C CNN
 F 2 "Diode_SMD:D_SOD-123" H 3000 4200 60  0001 C CNN
@@
 $EndComp
 $Comp
-L keyboard_parts:D D89
+L keyboard_parts:D D90
 U 1 1 5CBC246E
 P 6000 4200
-F 0 "D89" H 6050 4000 60  0000 R CNN
+F 0 "D90" H 6050 4000 60  0000 R CNN
 F 1 "D" V 6150 4150 60  0001 C CNN
 F 2 "Diode_SMD:D_SOD-123" H 6000 4200 60  0001 C CNN
@@
 $EndComp
 $Comp
-L keyboard_parts:D D90
+L keyboard_parts:D D91
 U 1 1 5CBC7EEC
 P 9000 4200
-F 0 "D90" H 9050 4000 60  0000 R CNN
+F 0 "D91" H 9050 4000 60  0000 R CNN
 F 1 "D" V 9150 4150 60  0001 C CNN
 F 2 "Diode_SMD:D_SOD-123" H 9000 4200 60  0001 C CNN
@@
 $EndComp
 $Comp
-L keyboard_parts:D D91
+L keyboard_parts:D D92
 U 1 1 5CBC7F4B
 P 9750 4200
-F 0 "D91" H 9800 4000 60  0000 R CNN
+F 0 "D92" H 9800 4000 60  0000 R CNN
 F 1 "D" V 9900 4150 60  0001 C CNN
 F 2 "Diode_SMD:D_SOD-123" H 9750 4200 60  0001 C CNN
@@
 $EndComp
 $Comp
-L keyboard_parts:D D92
+L keyboard_parts:D D93
 U 1 1 5CBC7FAA
 P 10500 4200
-F 0 "D92" H 10550 4000 60  0000 R CNN
+F 0 "D93" H 10550 4000 60  0000 R CNN
 F 1 "D" V 10650 4150 60  0001 C CNN
 F 2 "Diode_SMD:D_SOD-123" H 10500 4200 60  0001 C CNN
@@
 $EndComp
 $Comp
-L keyboard_parts:D D93
+L keyboard_parts:D D94
 U 1 1 5CBC8009
 P 11250 4200
-F 0 "D93" H 11300 4000 60  0000 R CNN
+F 0 "D94" H 11300 4000 60  0000 R CNN
 F 1 "D" V 11400 4150 60  0001 C CNN
 F 2 "Diode_SMD:D_SOD-123" H 11250 4200 60  0001 C CNN
@@
 $EndComp
 $Comp
-L keyboard_parts:SW_PUSH SW4,15
-U 1 1 5CBC8053
-P 12300 3550
-F 0 "SW4,15" H 12300 3700 50  0000 C CNN
-F 1 "UP" H 12300 3450 50  0000 C CNN
-F 2 "MX_SMK_2:MX_100" H 12300 3550 60  0001 C CNN
-F 3 "" H 12300 3550 60  0000 C CNN
-	1    12300 3550
-	1    0    0    -1
-$EndComp
-$Comp
-L keyboard_parts:D D84
-U 1 1 5CBC805A
-P 12000 3700
-F 0 "D84" H 12050 3500 60  0000 R CNN
-F 1 "D" V 12150 3650 60  0001 C CNN
-F 2 "Diode_SMD:D_SOD-123" H 12000 3700 60  0001 C CNN
-F 3 "" H 12000 3700 60  0000 C CNN
-	1    12000 3700
-	-1   0    0    1
-$EndComp
-$Comp
 L keyboard_parts:SW_PUSH SW5,15
 U 1 1 5CBC8061
@@
 $EndComp
 $Comp
-L keyboard_parts:D D94
+L keyboard_parts:D D95
 U 1 1 5CBC8068
 P 12000 4200
-F 0 "D94" H 12050 4000 60  0000 R CNN
+F 0 "D95" H 12050 4000 60  0000 R CNN
 F 1 "D" V 12150 4150 60  0001 C CNN
 F 2 "Diode_SMD:D_SOD-123" H 12000 4200 60  0001 C CNN
@@
 	-1   0    0    1
 $EndComp
-Wire Wire Line
-	12600 4050 12600 3550
 Connection ~ 12600 1550
 Wire Wire Line
@@
 Connection ~ 12600 3050
 Wire Wire Line
-	12600 3050 12600 2950
-Connection ~ 12600 3550
-Wire Wire Line
-	12600 3550 12600 3450
+	12600 3050 12600 3000
 $Comp
 L keyboard_parts:SW_PUSH SW0,16
@@
 $EndComp
 $Comp
-L keyboard_parts:D D95
+L keyboard_parts:D D96
 U 1 1 5CBD0B85
 P 12750 4200
-F 0 "D95" H 12800 4000 60  0000 R CNN
+F 0 "D96" H 12800 4000 60  0000 R CNN
 F 1 "D" V 12900 4150 60  0001 C CNN
 F 2 "Diode_SMD:D_SOD-123" H 12750 4200 60  0001 C CNN
@@
 Connection ~ 11250 3750
 Wire Wire Line
-	11250 3750 12000 3750
-Wire Wire Line
 	12750 4250 12000 4250
 Connection ~ 750  4250
@@
 	12000 4250 11250 4250
 Wire Wire Line
-	13350 3050 13350 3950
-Wire Wire Line
 	3000 4250 6000 4250
 Wire Wire Line
@@
 L keyboard_parts:SW_PUSH SW3,15-1
 U 1 1 5CE83AB0
-P 12300 2950
-F 0 "SW3,15-1" H 12300 3100 50  0000 C CNN
-F 1 "DEL" H 12300 2850 50  0000 C CNN
-F 2 "MX_SMK_2:MX_200" H 12300 2950 60  0001 C CNN
-F 3 "" H 12300 2950 60  0000 C CNN
-	1    12300 2950
+P 12300 3000
+F 0 "SW3,15-1" H 12300 3150 50  0000 C CNN
+F 1 "DEL" H 12300 2900 50  0000 C CNN
+F 2 "MX_SMK_2:MX_200" H 12300 3000 60  0001 C CNN
+F 3 "" H 12300 3000 60  0000 C CNN
+	1    12300 3000
 	1    0    0    -1
 $EndComp
-Connection ~ 12600 2950
-Wire Wire Line
-	12600 2950 12600 2550
-Wire Wire Line
-	12000 2950 12000 3050
 Connection ~ 12000 3050
 $Comp
@@
 	6000 3900 6000 3950
 $Comp
-L keyboard_parts:SW_PUSH SW4,15-1
-U 1 1 5CE61825
-P 12300 3450
-F 0 "SW4,15-1" H 12300 3600 50  0000 C CNN
-F 1 "Extra 1u" H 12300 3350 50  0000 C CNN
-F 2 "MX_SMK_2:MX_100" H 12300 3450 60  0001 C CNN
-F 3 "" H 12300 3450 60  0000 C CNN
-	1    12300 3450
-	1    0    0    -1
-$EndComp
-Connection ~ 12600 3450
-Wire Wire Line
-	12600 3450 12600 3050
-Wire Wire Line
-	12000 3450 12000 3550
-Connection ~ 12000 3550
-$Comp
-L dk_Trimmer-Potentiometers:TC33X-2-103E POT1
+L mad-cat-rescue:TC33X-2-103E-dk_Trimmer-Potentiometers POT1
 U 1 1 5CE8AE13
 P 8600 7300
@@
 	750  1950 750  2050
 Connection ~ 750  2050
+$Comp
+L keyboard_parts:SW_PUSH SW3,15-2
+U 1 1 5CE8D2C9
+P 12300 2950
+F 0 "SW3,15-2" H 12300 3100 50  0000 C CNN
+F 1 "DEL" H 12300 2850 50  0000 C CNN
+F 2 "MX_SMK_2:MX_100" H 12300 2950 60  0001 C CNN
+F 3 "" H 12300 2950 60  0000 C CNN
+	1    12300 2950
+	1    0    0    -1
+$EndComp
+Connection ~ 12600 2900
+Connection ~ 12000 3000
+Wire Wire Line
+	12000 3000 12000 3050
+Connection ~ 12600 3000
+Wire Wire Line
+	12000 2900 12000 2950
+Wire Wire Line
+	12600 2900 12600 2950
+Connection ~ 12000 2950
+Wire Wire Line
+	12000 2950 12000 3000
+Connection ~ 12600 2950
+Wire Wire Line
+	12600 2950 12600 3000
+Wire Wire Line
+	12600 2550 12600 2900
+Wire Wire Line
+	12750 3450 12750 3550
+$Comp
+L keyboard_parts:SW_PUSH SW3,15-3
+U 1 1 5CF1EE9B
+P 12300 2900
+F 0 "SW3,15-3" H 12300 3050 50  0000 C CNN
+F 1 "DEL" H 12300 2800 50  0000 C CNN
+F 2 "MX_SMK_2:MX_100" H 12300 2900 60  0001 C CNN
+F 3 "" H 12300 2900 60  0000 C CNN
+	1    12300 2900
+	1    0    0    -1
+$EndComp
+Connection ~ 12750 3550
+Wire Wire Line
+	13350 3050 13350 3450
+$Comp
+L keyboard_parts:SW_PUSH SW4,16-1
+U 1 1 5CE61825
+P 13050 3450
+F 0 "SW4,16-1" H 13050 3600 50  0000 C CNN
+F 1 "Extra 1u" H 13050 3350 50  0000 C CNN
+F 2 "MX_SMK_2:MX_100" H 13050 3450 60  0001 C CNN
+F 3 "" H 13050 3450 60  0000 C CNN
+	1    13050 3450
+	1    0    0    -1
+$EndComp
+$Comp
+L keyboard_parts:D D85
+U 1 1 5CBC805A
+P 12750 3700
+F 0 "D85" H 12800 3500 60  0000 R CNN
+F 1 "D" V 12900 3650 60  0001 C CNN
+F 2 "Diode_SMD:D_SOD-123" H 12750 3700 60  0001 C CNN
+F 3 "" H 12750 3700 60  0000 C CNN
+	1    12750 3700
+	-1   0    0    1
+$EndComp
+$Comp
+L keyboard_parts:SW_PUSH SW4,16
+U 1 1 5CBC8053
+P 13050 3550
+F 0 "SW4,16" H 13050 3700 50  0000 C CNN
+F 1 "UP" H 13050 3450 50  0000 C CNN
+F 2 "MX_SMK_2:MX_100" H 13050 3550 60  0001 C CNN
+F 3 "" H 13050 3550 60  0000 C CNN
+	1    13050 3550
+	1    0    0    -1
+$EndComp
+Connection ~ 13350 3450
+Wire Wire Line
+	13350 3450 13350 3550
+Connection ~ 13350 3550
+Wire Wire Line
+	13350 3550 13350 3950
+Wire Wire Line
+	12600 3050 12600 3450
+Wire Wire Line
+	11250 3750 12000 3750
+$Comp
+L keyboard_parts:D D84
+U 1 1 5D00187E
+P 12000 3700
+F 0 "D84" H 12050 3500 60  0000 R CNN
+F 1 "D" V 12150 3650 60  0001 C CNN
+F 2 "Diode_SMD:D_SOD-123" H 12000 3700 60  0001 C CNN
+F 3 "" H 12000 3700 60  0000 C CNN
+	1    12000 3700
+	-1   0    0    1
+$EndComp
+Connection ~ 12000 3750
+Wire Wire Line
+	12000 3750 12750 3750
+$Comp
+L keyboard_parts:SW_PUSH SW4,15
+U 1 1 5D001F00
+P 12300 3550
+F 0 "SW4,15" H 12300 3700 50  0000 C CNN
+F 1 "Extra 1u" H 12300 3450 50  0000 C CNN
+F 2 "MX_SMK_2:MX_100" H 12300 3550 60  0001 C CNN
+F 3 "" H 12300 3550 60  0000 C CNN
+	1    12300 3550
+	1    0    0    -1
+$EndComp
+Connection ~ 12600 3550
+Wire Wire Line
+	12600 3550 12600 4050
+$Comp
+L keyboard_parts:SW_PUSH SW4,15-1
+U 1 1 5D002C4E
+P 12300 3450
+F 0 "SW4,15-1" H 12300 3600 50  0000 C CNN
+F 1 "Extra 1u" H 12300 3350 50  0000 C CNN
+F 2 "MX_SMK_2:MX_100" H 12300 3450 60  0001 C CNN
+F 3 "" H 12300 3450 60  0000 C CNN
+	1    12300 3450
+	1    0    0    -1
+$EndComp
+Connection ~ 12600 3450
+Wire Wire Line
+	12600 3450 12600 3550
+Wire Wire Line
+	12000 3450 12000 3550
+Connection ~ 12000 3550
 $EndSCHEMATC
