File: pcb/mad cat.sch (KiCad schematic (older format))
At the start: 272 parts, among them J1 Conn_01x04, J2 Conn_02x03_Odd_Even, SW0,0 ESC, SW0,1 ESC/F1, SW0,10 F9, SW0,10-1 F10, SW0,11 F10, SW0,11-1 F11, SW0,12 F11, SW0,12-1 F12, SW0,13 F12/PRT, SW0,14 INS, SW0,15 HOME, SW0,16 PGUP, SW0,2 F1, SW0,2-1 F2, SW0,3 F2, SW0,3-1 F3, SW0,4 F3, SW0,4-1 F4, SW0,5 F4, SW0,5-1 F5, SW0,6 F5, SW0,6-1 F6, SW0,7 F6, SW0,7-1 F7, SW0,8 F7, SW0,8-1 F8, SW0,9 F8, SW0,9-1 F9, SW1,0 PF1, SW1,0-1 PF1, SW1,1 TILDE, SW1,10 9, SW1,11 0, SW1,12 -, SW1,13 =, SW1,14 BACKSPACE, SW1,14-1 S_BS_L, SW1,15 END, SW1,15-1 HOME, SW1,16 PGDN, SW1,16-1 PGUP, SW1,2 1, SW1,3 2, SW1,4 3, SW1,5 4, SW1,6 5, SW1,7 6, SW1,8 7, SW1,9 8, SW2,0 PF2, SW2,0-1 PF2, SW2,1 TAB, SW2,10 O, SW2,11 P, SW2,12 [, SW2,13 ], SW2,14 \\, SW2,15 S_BS_R, SW2,16 PRT, SW2,2 Q, SW2,3 W, SW2,4 E, SW2,5 R, SW2,6 T, SW2,7 Y, SW2,8 U, SW2,9 I, SW3,0 PF3, SW3,0-1 PF3, SW3,1 CAPS, SW3,1-1 ST_CAPS, SW3,10 L, SW3,11 COLONS, SW3,12 QUOTE, SW3,13 ISO_#, SW3,14 ENT, SW3,14-1 ISO_ENT, SW3,15 DEL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

Commit message: prepared for pcba
Parts:
- removed POT1: TC33X-2-103E, digikey-footprints:Trimpot_3.8mmx3.6mm_TC33X-2-103E, symbol mad-cat-rescue:TC33X-2-103E-dk_Trimmer-Potentiometers
- added LOGO1: MountingHole, logo:metamechs logo half, symbol Mechanical:MountingHole
- added POT1: TC33X-2-103E, digikey-footprints:Trimpot_3.8mmx3.6mm_TC33X-2-103E, symbol dk_Trimmer-Potentiometers:TC33X-2-103E
- C1, C10, C11, C12, C13, C2, C3, C4, C9: smt (none) -> C14663
- C5, C6: smt (none) -> C15849
- C7, C8: smt (none) -> C1653
- D1, D10, D11, D12, D13, D14, D15, D16, D17, D18, D19, D2, D20, D21, D22, D23, D24, D25, D26, D27, D28, D29, D3, D30, D31, D32, D33, D34, D35, D36, D37, D38, D39, D4, D40, D41, D42, D43, D44, D45, D46, D47, D48, D49, D5, D50, D51, D52, D53, D54, D55, D56, D57, D58, D59, D6, D60, D61, D62, D63, D64, D65, D66, D67, D68, D69, D7, D70, D71, D72, D73, D74, D75, D76, D77, D78, D79, D8, D80, D81, D82, D83, D84, D85, D86, D87, D88, D89, D9, D90, D91, D92, D93, D94, D95, D96, D97: symbol keyboard_parts:D -> mad-cat-rescue:D-keyboard_parts; smt (none) -> C81598
- R1, R2: symbol keyboard_parts:R -> mad-cat-rescue:R-keyboard_parts; smt (none) -> C23345
- R10, R6, R7, R8, R9: symbol keyboard_parts:R -> mad-cat-rescue:R-keyboard_parts; smt (none) -> C25804
- R5: symbol keyboard_parts:R -> mad-cat-rescue:R-keyboard_parts; smt (none) -> C23193
- RST1: footprint Button_Switch_SMD:SW_SPST_SKQG_WithStem -> crokto:TS-1187A-B-A-B; symbol keyboard_parts:SW_PUSH -> mad-cat-rescue:SW_PUSH-keyboard_parts; smt (none) -> C318884
- SW0,0, SW0,1, SW0,10, SW0,10-1, SW0,11, SW0,11-1, SW0,12, SW0,12-1, SW0,13, SW0,14, SW0,15, SW0,16, SW0,2, SW0,2-1, SW0,3, SW0,3-1, SW0,4, SW0,4-1, SW0,5, SW0,5-1, SW0,6, SW0,6-1, SW0,7, SW0,7-1, SW0,8, SW0,8-1, SW0,9, SW0,9-1, SW1,0, SW1,0-1, SW1,1, SW1,10, SW1,11, SW1,12, SW1,13, SW1,14, SW1,14-1, SW1,15, SW1,15-1, SW1,16, SW1,16-1, SW1,2, SW1,3, SW1,4, SW1,5, SW1,6, SW1,7, SW1,8, SW1,9, SW2,0, SW2,0-1, SW2,1, SW2,10, SW2,11, SW2,12, SW2,13, SW2,14, SW2,15, SW2,16, SW2,2, SW2,3, SW2,4, SW2,5, SW2,6, SW2,7, SW2,8, SW2,9, SW3,0, SW3,0-1, SW3,1, SW3,1-1, SW3,10, SW3,11, SW3,12, SW3,13, SW3,14, SW3,14-1, SW3,15, SW3,15-1, SW3,15-2, SW3,15-3, SW3,16, SW3,16-1, SW3,2, SW3,3, SW3,4, SW3,5, SW3,6, SW3,7, SW3,8, SW3,9, SW4,0, SW4,0-1, SW4,1, SW4,1-1, SW4,10, SW4,11, SW4,12, SW4,14, SW4,14-1, SW4,15, SW4,15-1, SW4,16, SW4,16-1, SW4,2, SW4,3, SW4,4, SW4,5, SW4,6, SW4,7, SW4,8, SW4,9, SW5,0, SW5,0-1, SW5,10, SW5,12, SW5,12-1, SW5,13, SW5,14, SW5,15, SW5,16, SW5,16-1, SW5,16-2, SW5,7, SW5,7-1: symbol keyboard_parts:SW_PUSH -> mad-cat-rescue:SW_PUSH-keyboard_parts
- SW4,13: footprint MX_SMK_2:MX_175 -> MX_SMK_2:MX_175_labeled; symbol keyboard_parts:SW_PUSH -> mad-cat-rescue:SW_PUSH-keyboard_parts
- SW4,13-1: footprint MX_SMK_2:MX_275 -> MX_SMK_2:MX_275_labeled; symbol keyboard_parts:SW_PUSH -> mad-cat-rescue:SW_PUSH-keyboard_parts
- SW5,1, SW5,11-1, SW5,3: footprint MX_SMK_2:MX_150 -> MX_SMK_2:MX_150_labeled; symbol keyboard_parts:SW_PUSH -> mad-cat-rescue:SW_PUSH-keyboard_parts
- SW5,1-1, SW5,2-1, SW5,3-1: footprint MX_SMK_2:MX_125 -> MX_SMK_2:MX_125_labeled; symbol keyboard_parts:SW_PUSH -> mad-cat-rescue:SW_PUSH-keyboard_parts
- SW5,11, SW5,2: footprint MX_SMK_2:MX_100 -> MX_SMK_2:MX_100_labeled; symbol keyboard_parts:SW_PUSH -> mad-cat-rescue:SW_PUSH-keyboard_parts
- U1: symbol keyboard_parts:ATMEGA32U4 -> mad-cat-rescue:ATMEGA32U4-keyboard_parts; smt (none) -> C44854
- Y1: footprint Crystal:Crystal_SMD_SeikoEpson_FA238-4Pin_3.2x2.5mm -> Crystal:Crystal_SMD_SeikoEpson_TSX3225-4Pin_3.2x2.5mm; smt (none) -> C89379
Connections:
- net GND: now also POT1.3 (CW)
- net at LED1.2 (A): now also POT1.2 (Wiper)
- net at R5.1: now also POT1.1 (CCW)

Commit message: edited LED circuit, flipped stabs
Parts:
- added ESD1: PRTR5V0U2X, Package_TO_SOT_SMD:SOT-143, symbol Power_Protection:PRTR5V0U2X
- added PTC1: 500mA, Fuse:Fuse_0805_2012Metric, symbol keyboard_parts:PTC
- C5: value 1u -> 10u; smt C15849 -> C19702
- R5: value 440 -> 510
- SW5,7: footprint MX_SMK_2:MX_625_stabflip -> MX_SMK_2:MX_625_nonflipped
- SW5,7-1: footprint MX_SMK_2:MX_600_stabflip_3 -> MX_SMK_2:MX_600_unflipped_3
Connections:
- net D+: now also ESD1.2 (I/O1)
- net D-: now also ESD1.3 (I/O2)
- net GND: now also ESD1.1 (GND); no longer POT1.3 (CW)
- net VCC: now also PTC1.2; no longer J1.4 (Pin_4)
- net at LED1.2 (A), POT1.2 (Wiper): now also POT1.1 (CCW)
- net at R5.1: now also POT1.3 (CW); no longer POT1.1 (CCW)
- new net vbus: ESD1.4 (VCC), J1.4 (Pin_4), PTC1.1
Other:
- moved on the sheet: C1, C10, C11, C12, C13, C2, C3, C4, C5, C6, C7, C8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

Commit message: new edge cuts
Parts:
- SW5,7: footprint MX_SMK_2:MX_625_nonflipped -> MX_SMK_2:MX_625_stabflip
- SW5,7-1: footprint MX_SMK_2:MX_600_unflipped_3 -> MX_SMK_2:MX_600_stabflip_3
Changed lines of the file:
@@
 F 0 "SW5,7" H 7350 5500 50  0000 C CNN
 F 1 "6.25U" H 7350 5250 50  0000 C CNN
-F 2 "MX_SMK_2:MX_625_nonflipped" H 7350 5350 60  0001 C CNN
+F 2 "MX_SMK_2:MX_625_stabflip" H 7350 5350 60  0001 C CNN
 F 3 "" H 7350 5350 60  0000 C CNN
 	1    7350 5350
@@
 F 0 "SW5,7-1" H 7350 5600 50  0000 C CNN
 F 1 "6U" H 7350 5350 50  0000 C CNN
-F 2 "MX_SMK_2:MX_600_unflipped_3" H 7350 5450 60  0001 C CNN
+F 2 "MX_SMK_2:MX_600_stabflip_3" H 7350 5450 60  0001 C CNN
 F 3 "" H 7350 5450 60  0000 C CNN
 	1    7350 5450
