File: pcb/backups/done but redoing.kicad_pcb (KiCad board)
At the start: 2 copper layers, 361.9 x 147 mm, 259 parts, among them J1 Conn_01x04, J2 Conn_02x03_Odd_Even, SW0,0 ESC, SW0,1 ESC/F1, SW0,10 F9, SW0,10-1 F10, SW0,11 F10, SW0,11-1 F11, SW0,12 F11, SW0,12-1 F12, SW0,13 F12/PRT, SW0,14 INS, SW0,15 HOME, SW0,16 PGUP, SW0,2 F1, SW0,2-1 F2, SW0,3 F2, SW0,3-1 F3, SW0,4 F3, SW0,4-1 F4, SW0,5 F4, SW0,5-1 F5, SW0,6 F5, SW0,6-1 F6, SW0,7 F6, SW0,7-1 F7, SW0,8 F7, SW0,8-1 F8, SW0,9 F8, SW0,9-1 F9, SW1,0 PF1, SW1,1 TILDE, SW1,10 9, SW1,11 0, SW1,12 -, SW1,13 =, SW1,14 BACKSPACE, SW1,14-1 S_BS_L, SW1,15 END, SW1,16 PGDN, SW1,2 1, SW1,3 2, SW1,4 3, SW1,5 4, SW1,6 5, SW1,7 6, SW1,8 7, SW1,9 8, SW2,0 PF2, SW2,1 TAB, SW2,10 O, SW2,11 P, SW2,12 [, SW2,13 ], SW2,14 \, SW2,15 S_BS_R, SW2,16 PRT, SW2,2 Q, SW2,3 W, SW2,4 E, SW2,5 R, SW2,6 T, SW2,7 Y, SW2,8 U, SW2,9 I, SW3,0 PF3, SW3,1 CAPS, SW3,1-1 ST_CAPS, SW3,10 L, SW3,11 COLONS, SW3,12 QUOTE, SW3,13 ISO_#, SW3,14 ENT, SW3,14-1 ISO_ENT, SW3,15 DEL, SW3,15-1 DEL, SW3,16 NP_ENT, SW3,16-1 1U_ENT, SW3,2 A, SW3,3 S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

Commit message: rebuilding pcb, adding switches to schematic
Parts:
- removed EC2-1: EC11E, keebs:EC11E
- removed SW3,15-1: DEL, MX_SMK_2:MX_SMK_200
- removed SW5,12-2: ALT, MX_SMK_2:MX_SMK_150
- removed SW5,7-2: 7 SPACE, MX_SMK_2:MX_SMK_700_stabflip
- added G***: LOGO, logo:metamechs logo half 2, B.Cu at (195.4, 111.1)
- added G***: LOGO, logo:metamechs logo half 2, F.Cu at (195.4, 111.1)
- C1, C10, C11, C12, C13, C2, C3, C4, C5, C6, C7, C8, C9: footprint Capacitor_SMD:C_0603_1608Metric -> Capacitor_SMD:C_0805_2012Metric
- R1, R10, R2, R5, R6, R7, R8, R9: footprint Resistor_SMD:R_0603_1608Metric -> Resistor_SMD:R_0805_2012Metric
- SW5,7-1: footprint MX_SMK_2:MX_SMK_625_stabflip -> MX_SMK_2:MX_SMK_625
- moved C13 242.9 mm to (350.8, 61.3), turned to 270 degrees
- moved C12 240.6 mm to (350.8, 65.7), turned to 270 degrees
- moved R10 236.5 mm to (347.5, 60.1), turned to 90 degrees
- moved R9 233.2 mm to (347.5, 67.0), turned to 90 degrees
- moved R7 167.6 mm to (8.25, 14.8), turned to 180 degrees
- moved R8 165.9 mm to (15.5, 13.2), turned to 180 degrees
- moved C10 164.6 mm to (6.25, 17.0), turned to 180 degrees
- moved C11 160.8 mm to (19.2, 13.2), turned to 180 degrees
- moved R2 4.92 mm to (120.2, 122.4)
- moved R1 4.77 mm to (121.6, 123.8)
- moved D10 4.00 mm to (206.0, 19.0)
- moved D11 4.00 mm to (232.4, 19.0)
- moved D12 4.00 mm to (251.4, 19.0)
- moved D13 4.00 mm to (270.5, 19.0)
- moved D3 4.00 mm to (61.2, 19.0)
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Connections:
- SW0,10-1 pad 1: /c10 -> Net-(D11-Pad2)
- SW0,10-1 pad 2: Net-(D11-Pad2) -> /c10
- SW0,11-1 pad 1: /c11 -> Net-(D12-Pad2)
- SW0,11-1 pad 2: Net-(D12-Pad2) -> /c11
- SW0,12-1 pad 1: /c12 -> Net-(D13-Pad2)
- SW0,12-1 pad 2: Net-(D13-Pad2) -> /c12
- SW0,2-1 pad 1: /c2 -> Net-(D3-Pad2)
- SW0,2-1 pad 2: Net-(D3-Pad2) -> /c2
- SW0,3-1 pad 1: /c3 -> Net-(D4-Pad2)
- SW0,3-1 pad 2: Net-(D4-Pad2) -> /c3
- SW0,4-1 pad 1: /c4 -> Net-(D5-Pad2)
- SW0,4-1 pad 2: Net-(D5-Pad2) -> /c4
- SW0,6-1 pad 1: /c6 -> Net-(D7-Pad2)
- SW0,6-1 pad 2: Net-(D7-Pad2) -> /c6
- SW0,7-1 pad 1: /c7 -> Net-(D8-Pad2)
- SW0,7-1 pad 2: Net-(D8-Pad2) -> /c7
- SW0,8-1 pad 1: /c8 -> Net-(D9-Pad2)
- SW0,8-1 pad 2: Net-(D9-Pad2) -> /c8
- SW3,1-1 pad 1: /c1 -> Net-(D53-Pad2)
- SW3,1-1 pad 2: Net-(D53-Pad2) -> /c1
- SW5,12-1 pad 1: /c12 -> Net-(D91-Pad2)
- SW5,12-1 pad 2: Net-(D91-Pad2) -> /c12
Routing:
- net GND: track 252.3 -> 704.5 mm, vias 3 -> 6
- net /enc+: track 263.0 -> 545.3 mm, vias 3 -> 6
- net /RES: track 0.00 -> 226.1 mm, vias 0 -> 2
- net /r5: track 148.5 -> 359.2 mm, vias 4 -> 6
- net /r0: track 317.5 -> 450.1 mm, vias 0 -> 4
- net /c13: track 190.8 -> 309.8 mm
- net VCC: track 224.8 -> 320.4 mm, vias 4 -> 9
- net Net-(LED1-Pad2): track 183.3 -> 276.0 mm, vias 2 -> 1
- net /c3: track 146.0 -> 232.7 mm, vias 0 -> 2
- net /r1: track 346.9 -> 423.4 mm
- net /c12: track 225.6 -> 279.6 mm
- net /c0: track 216.0 -> 267.4 mm
- net /enc-: track 466.9 -> 516.0 mm, vias 3 -> 4
- net /c1: track 261.0 -> 309.7 mm
- net /r2: track 398.0 -> 442.7 mm, vias 5 -> 6
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Other:
- net class gnd removed
- net class power: trace_width 0.381 -> 0.508; via_dia 1 -> 1.2; via_drill 0.5 -> 0.6
