File: pcb/backups/removing smk.kicad_pcb (KiCad board)
At the start: 2 copper layers, 361.9 x 147 mm, 262 parts, among them J1 Conn_01x04, J2 Conn_02x03_Odd_Even, SW0,0 ESC, SW0,1 ESC/F1, SW0,10 F9, SW0,10-1 F10, SW0,11 F10, SW0,11-1 F11, SW0,12 F11, SW0,12-1 F12, SW0,13 F12/PRT, SW0,14 INS, SW0,15 HOME, SW0,16 PGUP, SW0,2 F1, SW0,2-1 F2, SW0,3 F2, SW0,3-1 F3, SW0,4 F3, SW0,4-1 F4, SW0,5 F4, SW0,5-1 F5, SW0,6 F5, SW0,6-1 F6, SW0,7 F6, SW0,7-1 F7, SW0,8 F7, SW0,8-1 F8, SW0,9 F8, SW0,9-1 F9, SW1,0 PF1, SW1,1 TILDE, SW1,10 9, SW1,11 0, SW1,12 -, SW1,13 =, SW1,14 BACKSPACE, SW1,14-1 S_BS_L, SW1,15 END, SW1,16 PGDN, SW1,2 1, SW1,3 2, SW1,4 3, SW1,5 4, SW1,6 5, SW1,7 6, SW1,8 7, SW1,9 8, SW2,0 PF2, SW2,1 TAB, SW2,10 O, SW2,11 P, SW2,12 [, SW2,13 ], SW2,14 \, SW2,15 S_BS_R, SW2,16 PRT, SW2,2 Q, SW2,3 W, SW2,4 E, SW2,5 R, SW2,6 T, SW2,7 Y, SW2,8 U, SW2,9 I, SW3,0 PF3, SW3,1 CAPS, SW3,1-1 ST_CAPS, SW3,10 L, SW3,11 COLONS, SW3,12 QUOTE, SW3,13 ISO_#, SW3,14 ENT, SW3,14-1 ISO_ENT, SW3,15 DEL, SW3,15-1 DEL, SW3,16 NP_ENT, SW3,16-1 1U_ENT, SW3,2 A, SW3,3 S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

Commit message: redoing in mx only, adding trimpot for led
Parts:
- SW0,0, SW0,1, SW0,10, SW0,10-1, SW0,11, SW0,11-1, SW0,12, SW0,12-1, SW0,13, SW0,14, SW0,15, SW0,16, SW0,2, SW0,2-1, SW0,3, SW0,3-1, SW0,4, SW0,4-1, SW0,5, SW0,5-1, SW0,6, SW0,6-1, SW0,7, SW0,7-1, SW0,8, SW0,8-1, SW0,9, SW0,9-1, SW1,0, SW1,1, SW1,10, SW1,11, SW1,12, SW1,13, SW1,14-1, SW1,15, SW1,16, SW1,2, SW1,3, SW1,4, SW1,5, SW1,6, SW1,7, SW1,8, SW1,9, SW2,0, SW2,10, SW2,11, SW2,12, SW2,13, SW2,15, SW2,16, SW2,2, SW2,3, SW2,4, SW2,5, SW2,6, SW2,7, SW2,8, SW2,9, SW3,0, SW3,10, SW3,11, SW3,12, SW3,13, SW3,16-1, SW3,2, SW3,3, SW3,4, SW3,5, SW3,6, SW3,7, SW3,8, SW3,9, SW4,0, SW4,10, SW4,11, SW4,12, SW4,14, SW4,14-1, SW4,15, SW4,15-1, SW4,2, SW4,3, SW4,4, SW4,5, SW4,6, SW4,7, SW4,8, SW4,9, SW5,0, SW5,0-1, SW5,12, SW5,13-1, SW5,14, SW5,15, SW5,16, SW5,2: footprint MX_SMK_2:MX_100 -> MX_SMK_2:MX_SMK_100
- SW1,14, SW3,15, SW3,15-1, SW3,16, SW5,16-1: footprint MX_SMK_2:MX_200 -> MX_SMK_2:MX_SMK_200
- SW2,1, SW2,14, SW5,1, SW5,11, SW5,12-1, SW5,12-2, SW5,13, SW5,2-2, SW5,3: footprint MX_SMK_2:MX_150 -> MX_SMK_2:MX_SMK_150
- SW3,1, SW4,13: footprint MX_SMK_2:MX_175 -> MX_SMK_2:MX_SMK_175
- SW3,1-1, SW4,1-1, SW5,1-1, SW5,2-1, SW5,3-1: footprint MX_SMK_2:MX_125 -> MX_SMK_2:MX_SMK_125
- SW3,14, SW4,1: footprint MX_SMK_2:MX_225 -> MX_SMK_2:MX_SMK_225
- SW3,14-1: footprint MX_SMK_2:MX_ISO_stabflip -> MX_SMK_2:MX_SMK_ISO_stabflip
- SW4,13-1: footprint MX_SMK_2:MX_275 -> MX_SMK_2:MX_SMK_275
- SW5,7: footprint MX_SMK_2:MX_600_stabflip -> MX_SMK_2:MX_SMK_600_stabflip
- SW5,7-1: footprint MX_SMK_2:MX_625_stabflip -> MX_SMK_2:MX_SMK_625_stabflip
- SW5,7-2, SW5,7-3: footprint MX_SMK_2:MX_700_stabflip -> MX_SMK_2:MX_SMK_700_stabflip
- moved C11 2.43 mm to (14.6, 11.5)
- moved R8 2.42 mm to (14.6, 13.2)
- moved C1 1.43 mm to (113.8, 108.9)
- moved C10 0.70 mm to (6.80, 14.3)
Routing:
- net /c10: track 279.5 -> 252.9 mm
- net /c11: track 272.6 -> 252.2 mm
- net /c3: track 190.4 -> 209.9 mm, vias 1 -> 0
- net /RES: track 220.7 -> 239.3 mm, vias 4 -> 2
- net /enc-: track 503.7 -> 520.6 mm, vias 4 -> 6
- net /c7: track 172.6 -> 189.2 mm
- net /enc+: track 541.8 -> 525.9 mm, vias 4 -> 7
- net /c14: track 347.5 -> 361.3 mm
- net Net-(D32-Pad2): track 16.2 -> 27.9 mm
- net /c2: track 302.4 -> 291.8 mm
- net /c4: track 147.3 -> 157.5 mm
- net /c12: track 284.1 -> 275.3 mm
- net /r3: track 405.6 -> 398.1 mm, vias 4 -> 6
- net /r5: track 384.0 -> 376.9 mm, vias 6 -> 5
- net Net-(D51-Pad2): track 31.6 -> 38.6 mm
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Other:
- outline, holes or cut-outs redrawn
