File: pcb/backups/after stitch, going back.kicad_pcb (KiCad board)
At the start: 2 copper layers, 361.9 x 147 mm, 267 parts, among them J1 Conn_01x04, J2 Conn_02x03_Odd_Even, SW0,0 ESC, SW0,1 ESC/F1, SW0,10 F9, SW0,10-1 F10, SW0,11 F10, SW0,11-1 F11, SW0,12 F11, SW0,12-1 F12, SW0,13 F12/PRT, SW0,14 INS, SW0,15 HOME, SW0,16 PGUP, SW0,2 F1, SW0,2-1 F2, SW0,3 F2, SW0,3-1 F3, SW0,4 F3, SW0,4-1 F4, SW0,5 F4, SW0,5-1 F5, SW0,6 F5, SW0,6-1 F6, SW0,7 F6, SW0,7-1 F7, SW0,8 F7, SW0,8-1 F8, SW0,9 F8, SW0,9-1 F9, SW1,0 PF1, SW1,0-1 PF1, SW1,1 TILDE, SW1,10 9, SW1,11 0, SW1,12 -, SW1,13 =, SW1,14 BACKSPACE, SW1,14-1 S_BS_L, SW1,15 END, SW1,16 PGDN, SW1,2 1, SW1,3 2, SW1,4 3, SW1,5 4, SW1,6 5, SW1,7 6, SW1,8 7, SW1,9 8, SW2,0 PF2, SW2,0-1 PF2, SW2,1 TAB, SW2,10 O, SW2,11 P, SW2,12 [, SW2,13 ], SW2,14 \, SW2,15 S_BS_R, SW2,16 PRT, SW2,2 Q, SW2,3 W, SW2,4 E, SW2,5 R, SW2,6 T, SW2,7 Y, SW2,8 U, SW2,9 I, SW3,0 PF3, SW3,0-1 PF3, SW3,1 CAPS, SW3,1-1 ST_CAPS, SW3,10 L, SW3,11 COLONS, SW3,12 QUOTE, SW3,13 ISO_#, SW3,14 ENT, SW3,14-1 ISO_ENT, SW3,15 DEL, SW3,15-1 DEL, SW3,16 NP_ENT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

Commit message: reverting vias
Routing:
- net GND: vias 5723 -> 5726
Changed lines of the file:
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@@
     (thickness 1.6)
     (drawings 76)
-    (tracks 6971)
+    (tracks 6974)
     (zones 0)
     (modules 267)
@@
   (via (at 199.6 100.2) (size 0.6) (drill 0.3) (layers F.Cu B.Cu) (net 1))
   (via (at 285.7 100.5) (size 0.6) (drill 0.3) (layers F.Cu B.Cu) (net 1))
+  (via (at 16.372619 37.893545) (size 0.6) (drill 0.3) (layers F.Cu B.Cu) (net 1))
+  (via (at 19.380904 87.995857) (size 0.6) (drill 0.3) (layers F.Cu B.Cu) (net 1))
+  (via (at 171.584308 51.444886) (size 0.6) (drill 0.3) (layers F.Cu B.Cu) (net 1))
   (segment (start 117.2875 117.5) (end 117.368629 117.5) (width 0.381) (layer B.Cu) (net 2) (status 30))
   (via (at 118.134314 116.734314) (size 1) (drill 0.5) (layers F.Cu B.Cu) (net 2))
