File: pcb/backups/pre-stitch again.kicad_pcb (KiCad board)
At the start: 2 copper layers, 361.9 x 147 mm, 262 parts, among them J1 Conn_01x04, J2 Conn_02x03_Odd_Even, SW0,0 ESC, SW0,1 ESC/F1, SW0,10 F9, SW0,10-1 F10, SW0,11 F10, SW0,11-1 F11, SW0,12 F11, SW0,12-1 F12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

Commit message: little updates
Routing:
- net /c9: track 179.7 -> 186.1 mm
- net Net-(R5-Pad2): track 265.9 -> 263.7 mm
Other:
- outline, holes or cut-outs redrawn
