File: pcb/backups/pre proto 5.kicad_pcb (KiCad board)
At the start: 2 copper layers, 361.9 x 143 mm, 275 parts, among them J1 Conn_01x04, J2 Conn_02x03_Odd_Even, SW0,0 ESC, SW0,1 ESC/F1, SW0,10 F9, SW0,10-1 F10, SW0,11 F10, SW0,11-1 F11, SW0,12 F11, SW0,12-1 F12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

Commit message: little updates
Parts:
- D1, D10, D11, D12, D13, D14, D15, D16, D17, D18, D19, D2, D20, D21, D22, D23, D24, D25, D26, D27, D28, D29, D3, D30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: footprint keebs:D_SOD-123proto -> Diode_SMD:D_SOD-123
Routing:
- net GND: track 298.2 -> 301.0 mm, vias 84 -> 85
