File: pcb/backups/SENT TO JLC 2.kicad_pcb (KiCad board)
At the start: 2 copper layers, 361.9 x 143 mm, 272 parts, among them J1 Conn_01x04, J2 Conn_02x03_Odd_Even, SW0,0 ESC, SW0,1 ESC/F1, SW0,10 F9, SW0,10-1 F10, SW0,11 F10, SW0,11-1 F11, SW0,12 F11, SW0,12-1 F12, SW0,13 F12/PRT, SW0,14 INS, SW0,15 HOME, SW0,16 PGUP, SW0,2 F1, SW0,2-1 F2, SW0,3 F2, SW0,3-1 F3, SW0,4 F3, SW0,4-1 F4, SW0,5 F4, SW0,5-1 F5, SW0,6 F5, SW0,6-1 F6, SW0,7 F6, SW0,7-1 F7, SW0,8 F7, SW0,8-1 F8, SW0,9 F8, SW0,9-1 F9, SW1,0 PF1, SW1,0-1 PF1, SW1,1 TILDE, SW1,10 9, SW1,11 0, SW1,12 -, SW1,13 =, SW1,14 BACKSPACE, SW1,14-1 S_BS_L, SW1,15 END, SW1,15-1 HOME, SW1,16 PGDN, SW1,16-1 PGUP, SW1,2 1, SW1,3 2, SW1,4 3, SW1,5 4, SW1,6 5, SW1,7 6, SW1,8 7, SW1,9 8, SW2,0 PF2, SW2,0-1 PF2, SW2,1 TAB, SW2,10 O, SW2,11 P, SW2,12 [, SW2,13 ], SW2,14 \, SW2,15 S_BS_R, SW2,16 PRT, SW2,2 Q, SW2,3 W, SW2,4 E, SW2,5 R, SW2,6 T, SW2,7 Y, SW2,8 U, SW2,9 I, SW3,0 PF3, SW3,0-1 PF3, SW3,1 CAPS, SW3,1-1 ST_CAPS, SW3,10 L, SW3,11 COLONS, SW3,12 QUOTE, SW3,13 ISO_#, SW3,14 ENT, SW3,14-1 ISO_ENT, SW3,15 DEL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

Commit message: updated switch rotations
Parts:
- removed SW5,7-1: 6U, MX_SMK_2:MX_600_stabflip3
- added G***: LOGO, logo:metamechs logo half, B.Cu at (201.0, 111.1)
- added G***: LOGO, logo:metamechs logo half, F.Cu at (201.0, 111.1)
- added SW5,7-2: 6U OC, MX_SMK_2:MX_100, F.Cu at (168.3, 111.1)
- added SW5,7-3: 6U, MX_SMK_2:MX_600_stabflip, F.Cu at (158.8, 111.1)
- LED1: footprint crokto:LED_0805_lightpipe -> keebs:LED_0805_lightpipe
- turned SW2,15 to 90 degrees
- turned SW4,1-1 to 90 degrees
Routing:
- net Net-(D90-Pad2): track 26.0 -> 43.1 mm
- net /r5: track 405.6 -> 415.5 mm
- net /c1: track 286.7 -> 295.3 mm
- net /c15: track 420.7 -> 427.2 mm
- net Net-(D50-Pad2): track 10.3 -> 5.30 mm
- net /c7: track 175.3 -> 171.5 mm
- net Net-(D70-Pad2): track 20.7 -> 20.1 mm
- net GND: vias 71 -> 3395
