File: pcb/daughterboard/daughterboard.kicad_pcb (KiCad board)
At the start: 2 copper layers, 22 x 19 mm, 11 parts, among them J1 Conn_01x04

Commit message: prepared for pcba
Parts:
- removed G***: LOGO, logo:logo tiny vert
- added J2: Conn_01x04, Connector_JST:JST_SH_SM04B-SRSS-TB_1x04-1MP_P1.00mm_Horizontal, F.Cu at (17.7, 11.5)
- F1: value PTC -> 500mA
- moved R1 0.40 mm to (17.0, 7.10)
Routing:
- net GND: track 4.53 -> 33.4 mm
- net VCC: track 12.5 -> 30.7 mm, vias 0 -> 2
- net /d+: track 18.5 -> 28.8 mm, vias 0 -> 2
- net /d-: track 19.6 -> 26.6 mm

Commit message: edited LED circuit, flipped stabs
Parts:
- removed C1: 10u, Capacitor_SMD:C_0603_1608Metric
- removed D1: PRTR5V0U2X, Package_TO_SOT_SMD:SOT-143
- removed F1: 500mA, Fuse:Fuse_0805_2012Metric
- removed J2: Conn_01x04, Connector_JST:JST_SH_SM04B-SRSS-TB_1x04-1MP_P1.00mm_Horizontal
- J1: footprint Connector_PinHeader_2.00mm:PinHeader_1x04_P2.00mm_Vertical -> Connector_JST:JST_SH_SM04B-SRSS-TB_1x04-1MP_P1.00mm_Horizontal
- moved J1 0.61 mm to (4.00, 11.0), turned to 180 degrees
- moved R2 0.10 mm to (4.40, 6.80)
Connections:
- J1 pad 4: VCC -> /vbus
Routing:
- net VCC: track 30.7 -> 0.00 mm, vias 2 -> 0
- net /d+: track 28.8 -> 14.5 mm, vias 2 -> 0
- net GND: track 33.4 -> 47.3 mm, vias 4 -> 0
- net /vbus: track 13.5 -> 23.9 mm
- net /d-: track 26.6 -> 17.8 mm
